File: PCB_layout/mechanical.sch (KiCad schematic (older format))
At the start: 11 parts, among them U7 Sensor_O2_US

Commit message: PCB layout, WIP
Parts:
- removed HB45, HB46: mtg_hole_3mm_small, AA_vayu:MountingHole_3.2mm_M3, symbol AA_vayuO2_symbols:SCREW
- removed HB47, HB48, HB53, HB54: mtg_hole_3mm, AA_vayu:MountingHole_3.2mm_M3_Pad_Via, symbol AA_vayuO2_symbols:SCREW
- added CN19: Conn_O2_5V, AA_vayu:JST_EH_B2B-EH-A_1x02_P2.50mm_Vertical, symbol AA_vayuO2_symbols:Conn_01x02
- added MB1, MB2, MB3, MB4, MB5, MB6: Mouse_Bite, AA_vayu:mouse-bite-2.54mm-slot_OSH, symbol AA_vayuO2_symbols:Mouse_Bite
- added U10: Sensor_O2_US_narrow, AA_vayu:Sensor_O2_US_narrow, symbol AA_vayuO2_symbols:Sensor_O2_US
- HB1: renamed from HB49; footprint AA_vayu:MountingHole_3.2mm_M3 -> AA_vayu:MountingHole_3.2mm_M3_Pad_Via
- HB2: renamed from HB50; footprint AA_vayu:MountingHole_3.2mm_M3 -> AA_vayu:MountingHole_3.2mm_M3_Pad_Via
- HB3: renamed from HB51; footprint AA_vayu:MountingHole_3.2mm_M3 -> AA_vayu:MountingHole_3.2mm_M3_Pad_Via
- HB4: renamed from HB52; footprint AA_vayu:MountingHole_3.2mm_M3 -> AA_vayu:MountingHole_3.2mm_M3_Pad_Via
Connections:
- new net 5V: CN19.1 (Pin_1)
- new net GND: CN19.2 (Pin_2)
Other:
- note added: "5V Supply for O2 Sensor"
- note added: "ALTERNATE MECHANICAL FOOTPRINT\nFOR ULTRASONIC O2 SENSOR"
- note added: "MOUSE BITES"
- note removed: "<- 0.575" ->"
- note removed: "<- 1.35" ->"
- note removed: "<- 2.8" ->"
- note removed: "<- 6.0" ->"
- note removed: "<- 6.1" ->"
- moved on the sheet: U7
Changed lines of the file:
@@
 $EndDescr
 $Comp
-L AA_vayuO2_symbols:SCREW HB45
-U 1 1 5A4A80D0
-P 1700 3750
-F 0 "HB45" V 1700 3672 40  0000 R CNN
-F 1 "mtg_hole_3mm_small" H 1700 3850 40  0001 C CNN
-F 2 "AA_vayu:MountingHole_3.2mm_M3" H 1778 3713 60  0001 L CNN
-F 3 "" H 1700 3750 60  0000 C CNN
-F 4 "Value" H 1700 3750 50  0001 C CNN "manf#"
-	1    1700 3750
-	0    -1   -1   0
-$EndComp
-$Comp
-L AA_vayuO2_symbols:SCREW HB46
-U 1 1 5A4A8341
-P 3200 3750
-F 0 "HB46" V 3200 3672 40  0000 R CNN
-F 1 "mtg_hole_3mm_small" H 3200 3850 40  0001 C CNN
-F 2 "AA_vayu:MountingHole_3.2mm_M3" H 3278 3713 60  0001 L CNN
-F 3 "" H 3200 3750 60  0000 C CNN
-F 4 "Value" H 3200 3750 50  0001 C CNN "manf#"
-	1    3200 3750
-	0    1    1    0
-$EndComp
-$Comp
-L AA_vayuO2_symbols:SCREW HB47
-U 1 1 5A4A8811
-P 1750 4250
-F 0 "HB47" V 1750 4172 40  0000 R CNN
-F 1 "mtg_hole_3mm" H 1750 4350 40  0001 C CNN
-F 2 "AA_vayu:MountingHole_3.2mm_M3_Pad_Via" H 1828 4213 60  0001 L CNN
-F 3 "" H 1750 4250 60  0000 C CNN
-F 4 "Value" H 1750 4250 50  0001 C CNN "manf#"
-	1    1750 4250
-	0    -1   -1   0
-$EndComp
-$Comp
-L AA_vayuO2_symbols:SCREW HB48
-U 1 1 5A4A8818
-P 3150 4250
-F 0 "HB48" V 3150 4172 40  0000 R CNN
-F 1 "mtg_hole_3mm" H 3150 4350 40  0001 C CNN
-F 2 "AA_vayu:MountingHole_3.2mm_M3_Pad_Via" H 3228 4213 60  0001 L CNN
-F 3 "" H 3150 4250 60  0000 C CNN
-F 4 "Value" H 3150 4250 50  0001 C CNN "manf#"
-	1    3150 4250
-	0    1    1    0
-$EndComp
-$Comp
-L AA_vayuO2_symbols:SCREW HB53
-U 1 1 5A4A8943
-P 1750 5250
-F 0 "HB53" V 1750 5172 40  0000 R CNN
-F 1 "mtg_hole_3mm" H 1750 5350 40  0001 C CNN
-F 2 "AA_vayu:MountingHole_3.2mm_M3_Pad_Via" H 1828 5213 60  0001 L CNN
-F 3 "" H 1750 5250 60  0000 C CNN
-F 4 "Value" H 1750 5250 50  0001 C CNN "manf#"
-	1    1750 5250
-	0    -1   -1   0
-$EndComp
-$Comp
-L AA_vayuO2_symbols:SCREW HB54
-U 1 1 5A4A894A
-P 3150 5250
-F 0 "HB54" V 3150 5172 40  0000 R CNN
-F 1 "mtg_hole_3mm" H 3150 5350 40  0001 C CNN
-F 2 "AA_vayu:MountingHole_3.2mm_M3_Pad_Via" H 3228 5213 60  0001 L CNN
-F 3 "" H 3150 5250 60  0000 C CNN
-F 4 "Value" H 3150 5250 50  0001 C CNN "manf#"
-	1    3150 5250
-	0    1    1    0
-$EndComp
-Text Notes 2300 3775 0    40   ~ 0
-<- 6.1" ->
-Text Notes 2300 5275 0    40   ~ 0
-<- 6.0" ->
-Text Notes 1775 4950 1    40   ~ 0
-<- 6.0" ->
-Text Notes 1700 4225 1    40   ~ 0
-<- 1.35" ->
-Wire Notes Line
-	1600 3650 3300 3650
-Wire Notes Line
-	3300 3650 3300 5850
-Wire Notes Line
-	3300 5850 1600 5850
-Wire Notes Line
-	1600 5850 1600 3650
-$Comp
-L AA_vayuO2_symbols:SCREW HB49
+L AA_vayuO2_symbols:SCREW HB1
 U 1 1 5A736F2B
 P 4350 4350
-F 0 "HB49" V 4350 4272 40  0000 R CNN
+F 0 "HB1" V 4350 4272 40  0000 R CNN
 F 1 "mtg_hole_3mm" H 4350 4450 40  0001 C CNN
-F 2 "AA_vayu:MountingHole_3.2mm_M3" H 4428 4313 60  0001 L CNN
+F 2 "AA_vayu:MountingHole_3.2mm_M3_Pad_Via" H 4428 4313 60  0001 L CNN
 F 3 "" H 4350 4350 60  0000 C CNN
 F 4 "Value" H 4350 4350 50  0001 C CNN "manf#"
@@
 $EndComp
 $Comp
-L AA_vayuO2_symbols:SCREW HB50
+L AA_vayuO2_symbols:SCREW HB2
 U 1 1 5A736F32
 P 5150 4350
-F 0 "HB50" V 5150 4272 40  0000 R CNN
+F 0 "HB2" V 5150 4272 40  0000 R CNN
 F 1 "mtg_hole_3mm" H 5150 4450 40  0001 C CNN
-F 2 "AA_vayu:MountingHole_3.2mm_M3" H 5228 4313 60  0001 L CNN
+F 2 "AA_vayu:MountingHole_3.2mm_M3_Pad_Via" H 5228 4313 60  0001 L CNN
 F 3 "" H 5150 4350 60  0000 C CNN
 F 4 "Value" H 5150 4350 50  0001 C CNN "manf#"
@@
 $EndComp
 $Comp
-L AA_vayuO2_symbols:SCREW HB51
+L AA_vayuO2_symbols:SCREW HB3
 U 1 1 5A736F39
 P 4350 5150
-F 0 "HB51" V 4350 5072 40  0000 R CNN
+F 0 "HB3" V 4350 5072 40  0000 R CNN
 F 1 "mtg_hole_3mm" H 4350 5250 40  0001 C CNN
-F 2 "AA_vayu:MountingHole_3.2mm_M3" H 4428 5113 60  0001 L CNN
+F 2 "AA_vayu:MountingHole_3.2mm_M3_Pad_Via" H 4428 5113 60  0001 L CNN
 F 3 "" H 4350 5150 60  0000 C CNN
 F 4 "Value" H 4350 5150 50  0001 C CNN "manf#"
@@
 $EndComp
 $Comp
-L AA_vayuO2_symbols:SCREW HB52
+L AA_vayuO2_symbols:SCREW HB4
 U 1 1 5A736F40
 P 5150 5150
-F 0 "HB52" V 5150 5072 40  0000 R CNN
+F 0 "HB4" V 5150 5072 40  0000 R CNN
 F 1 "mtg_hole_3mm" H 5150 5250 40  0001 C CNN
-F 2 "AA_vayu:MountingHole_3.2mm_M3" H 5228 5113 60  0001 L CNN
+F 2 "AA_vayu:MountingHole_3.2mm_M3_Pad_Via" H 5228 5113 60  0001 L CNN
 F 3 "" H 5150 5150 60  0000 C CNN
 F 4 "Value" H 5150 5150 50  0001 C CNN "manf#"
@@
 	0    1    1    0
 $EndComp
-Text Notes 4550 5250 0    40   ~ 0
-<- 2.8" ->
-Text Notes 4375 4950 1    40   ~ 0
-<- 2.8" ->
 Wire Notes Line
 	3900 3650 5600 3650
@@
 Wire Notes Line
 	3900 5850 3900 3650
-Wire Notes Line
-	4750 4650 4750 4850
-Wire Notes Line
-	2350 4750 2550 4750
-Wire Notes Line
-	2450 4650 2450 4850
-Text Notes 5300 4775 1    40   ~ 0
-<- 0.575" ->
-Wire Notes Line
-	4650 4750 5225 4750
 $Comp
 L AA_vayuO2_symbols:Sensor_O2_US U7
 U 1 1 61775E18
-P 7275 4050
-F 0 "U7" H 6925 4200 40  0000 C CNN
-F 1 "Sensor_O2_US" H 7475 4200 40  0000 C CNN
-F 2 "AA_vayu:Sensor_O2_US" H 7275 4050 40  0001 C CNN
-F 3 "" H 7275 4050 40  0001 C CNN
-	1    7275 4050
+P 7275 2650
+F 0 "U7" H 6925 2800 40  0000 C CNN
+F 1 "Sensor_O2_US" H 7475 2800 40  0000 C CNN
+F 2 "AA_vayu:Sensor_O2_US" H 7275 2650 40  0001 C CNN
+F 3 "" H 7275 2650 40  0001 C CNN
+	1    7275 2650
 	1    0    0    -1
 $EndComp
-Text Notes 6850 4475 0    50   ~ 10
+Text Notes 6850 3050 0    50   ~ 10
 MECHANICAL FOOTPRINT\nFOR ULTRASONIC O2 SENSOR
+$Comp
+L AA_vayuO2_symbols:Conn_01x02 CN19
+U 1 1 6167392A
+P 7625 1875
+F 0 "CN19" H 7750 1900 50  0000 L CNN
+F 1 "Conn_O2_5V" H 7750 1800 50  0000 L CNN
+F 2 "AA_vayu:JST_EH_B2B-EH-A_1x02_P2.50mm_Vertical" H 7625 1875 50  0001 C CNN
+F 3 "" H 7625 1875 50  0001 C CNN
+	1    7625 1875
+	1    0    0    -1
+$EndComp
+Wire Wire Line
+	7425 1875 7100 1875
+Wire Wire Line
+	7425 1975 7100 1975
+Text HLabel 7100 1875 0    40   Input ~ 0
+5V
+Text HLabel 7100 1975 0    40   Input ~ 0
+GND
+$Comp
+L AA_vayuO2_symbols:Mouse_Bite MB1
+U 1 1 61695C97
+P 7050 5725
+F 0 "MB1" H 7000 5725 40  0000 L CNN
+F 1 "Mouse_Bite" H 7050 5850 30  0001 C CNN
+F 2 "AA_vayu:mouse-bite-2.54mm-slot_OSH" H 7050 5725 60  0001 C CNN
+F 3 "" H 7050 5725 60  0000 C CNN
+	1    7050 5725
+	1    0    0    -1
+$EndComp
+$Comp
+L AA_vayuO2_symbols:Mouse_Bite MB2
+U 1 1 616967E9
+P 7650 5725
+F 0 "MB2" H 7600 5725 40  0000 L CNN
+F 1 "Mouse_Bite" H 7650 5850 30  0001 C CNN
+F 2 "AA_vayu:mouse-bite-2.54mm-slot_OSH" H 7650 5725 60  0001 C CNN
+F 3 "" H 7650 5725 60  0000 C CNN
+	1    7650 5725
+	1    0    0    -1
+$EndComp
+$Comp
+L AA_vayuO2_symbols:Mouse_Bite MB3
+U 1 1 61696DDA
+P 8250 5725
+F 0 "MB3" H 8200 5725 40  0000 L CNN
+F 1 "Mouse_Bite" H 8250 5850 30  0001 C CNN
+F 2 "AA_vayu:mouse-bite-2.54mm-slot_OSH" H 8250 5725 60  0001 C CNN
+F 3 "" H 8250 5725 60  0000 C CNN
+	1    8250 5725
+	1    0    0    -1
+$EndComp
+$Comp
+L AA_vayuO2_symbols:Mouse_Bite MB4
+U 1 1 61698785
+P 8775 5350
+F 0 "MB4" H 8725 5350 40  0000 L CNN
+F 1 "Mouse_Bite" H 8775 5475 30  0001 C CNN
+F 2 "AA_vayu:mouse-bite-2.54mm-slot_OSH" H 8775 5350 60  0001 C CNN
+F 3 "" H 8775 5350 60  0000 C CNN
+	1    8775 5350
+	0    -1   -1   0
+$EndComp
+$Comp
+L AA_vayuO2_symbols:Mouse_Bite MB5
+U 1 1 61698831
+P 8775 4750
+F 0 "MB5" H 8725 4750 40  0000 L CNN
+F 1 "Mouse_Bite" H 8775 4875 30  0001 C CNN
+F 2 "AA_vayu:mouse-bite-2.54mm-slot_OSH" H 8775 4750 60  0001 C CNN
+F 3 "" H 8775 4750 60  0000 C CNN
+	1    8775 4750
+	0    -1   -1   0
+$EndComp
+$Comp
+L AA_vayuO2_symbols:Mouse_Bite MB6
+U 1 1 6169883B
+P 8775 4150
+F 0 "MB6" H 8725 4150 40  0000 L CNN
+F 1 "Mouse_Bite" H 8775 4275 30  0001 C CNN
+F 2 "AA_vayu:mouse-bite-2.54mm-slot_OSH" H 8775 4150 60  0001 C CNN
+F 3 "" H 8775 4150 60  0000 C CNN
+	1    8775 4150
+	0    -1   -1   0
+$EndComp
+Text Notes 7425 6000 0    40   ~ 8
+MOUSE BITES
+Text Notes 6850 1650 0    50   ~ 10
+5V Supply for O2 Sensor
+$Comp
+L AA_vayuO2_symbols:Sensor_O2_US U10
+U 1 1 616B2CD7
+P 7275 3550
+F 0 "U10" H 6925 3700 40  0000 C CNN
+F 1 "Sensor_O2_US_narrow" H 7475 3700 40  0000 C CNN
+F 2 "AA_vayu:Sensor_O2_US_narrow" H 7275 3550 40  0001 C CNN
+F 3 "" H 7275 3550 40  0001 C CNN
+	1    7275 3550
+	1    0    0    -1
+$EndComp
+Text Notes 6850 3925 0    50   ~ 10
+ALTERNATE MECHANICAL FOOTPRINT\nFOR ULTRASONIC O2 SENSOR
 $EndSCHEMATC

Commit message: BOM, WIP
Parts:
- removed MB1, MB2, MB3, MB4, MB5, MB6: Mouse_Bite, AA_vayu:mouse-bite-2.54mm-slot_OSH, symbol AA_vayuO2_symbols:Mouse_Bite
- removed U10: Sensor_O2_US_narrow, AA_vayu:Sensor_O2_US_narrow, symbol AA_vayuO2_symbols:Sensor_O2_US
- removed U7: Sensor_O2_US, AA_vayu:Sensor_O2_US, symbol AA_vayuO2_symbols:Sensor_O2_US
Other:
- note removed: "MOUSE BITES"
Changed lines of the file:
@@
 	3900 5850 3900 3650
 $Comp
-L AA_vayuO2_symbols:Sensor_O2_US U7
+L AA_vayuO2_symbols:Sensor_O2_US #U7
 U 1 1 61775E18
 P 7275 2650
-F 0 "U7" H 6925 2800 40  0000 C CNN
+F 0 "#U7" H 6925 2800 40  0000 C CNN
 F 1 "Sensor_O2_US" H 7475 2800 40  0000 C CNN
 F 2 "AA_vayu:Sensor_O2_US" H 7275 2650 40  0001 C CNN
@@
 Text HLabel 7100 1975 0    40   Input ~ 0
 GND
-$Comp
-L AA_vayuO2_symbols:Mouse_Bite MB1
-U 1 1 61695C97
-P 7050 5725
-F 0 "MB1" H 7000 5725 40  0000 L CNN
-F 1 "Mouse_Bite" H 7050 5850 30  0001 C CNN
-F 2 "AA_vayu:mouse-bite-2.54mm-slot_OSH" H 7050 5725 60  0001 C CNN
-F 3 "" H 7050 5725 60  0000 C CNN
-	1    7050 5725
-	1    0    0    -1
-$EndComp
-$Comp
-L AA_vayuO2_symbols:Mouse_Bite MB2
-U 1 1 616967E9
-P 7650 5725
-F 0 "MB2" H 7600 5725 40  0000 L CNN
-F 1 "Mouse_Bite" H 7650 5850 30  0001 C CNN
-F 2 "AA_vayu:mouse-bite-2.54mm-slot_OSH" H 7650 5725 60  0001 C CNN
-F 3 "" H 7650 5725 60  0000 C CNN
-	1    7650 5725
-	1    0    0    -1
-$EndComp
-$Comp
-L AA_vayuO2_symbols:Mouse_Bite MB3
-U 1 1 61696DDA
-P 8250 5725
-F 0 "MB3" H 8200 5725 40  0000 L CNN
-F 1 "Mouse_Bite" H 8250 5850 30  0001 C CNN
-F 2 "AA_vayu:mouse-bite-2.54mm-slot_OSH" H 8250 5725 60  0001 C CNN
-F 3 "" H 8250 5725 60  0000 C CNN
-	1    8250 5725
-	1    0    0    -1
-$EndComp
-$Comp
-L AA_vayuO2_symbols:Mouse_Bite MB4
-U 1 1 61698785
-P 8775 5350
-F 0 "MB4" H 8725 5350 40  0000 L CNN
-F 1 "Mouse_Bite" H 8775 5475 30  0001 C CNN
-F 2 "AA_vayu:mouse-bite-2.54mm-slot_OSH" H 8775 5350 60  0001 C CNN
-F 3 "" H 8775 5350 60  0000 C CNN
-	1    8775 5350
-	0    -1   -1   0
-$EndComp
-$Comp
-L AA_vayuO2_symbols:Mouse_Bite MB5
-U 1 1 61698831
-P 8775 4750
-F 0 "MB5" H 8725 4750 40  0000 L CNN
-F 1 "Mouse_Bite" H 8775 4875 30  0001 C CNN
-F 2 "AA_vayu:mouse-bite-2.54mm-slot_OSH" H 8775 4750 60  0001 C CNN
-F 3 "" H 8775 4750 60  0000 C CNN
-	1    8775 4750
-	0    -1   -1   0
-$EndComp
-$Comp
-L AA_vayuO2_symbols:Mouse_Bite MB6
-U 1 1 6169883B
-P 8775 4150
-F 0 "MB6" H 8725 4150 40  0000 L CNN
-F 1 "Mouse_Bite" H 8775 4275 30  0001 C CNN
-F 2 "AA_vayu:mouse-bite-2.54mm-slot_OSH" H 8775 4150 60  0001 C CNN
-F 3 "" H 8775 4150 60  0000 C CNN
-	1    8775 4150
-	0    -1   -1   0
-$EndComp
-Text Notes 7425 6000 0    40   ~ 8
-MOUSE BITES
 Text Notes 6850 1650 0    50   ~ 10
 5V Supply for O2 Sensor
 $Comp
-L AA_vayuO2_symbols:Sensor_O2_US U10
+L AA_vayuO2_symbols:Sensor_O2_US #U10
 U 1 1 616B2CD7
 P 7275 3550
-F 0 "U10" H 6925 3700 40  0000 C CNN
+F 0 "#U10" H 6925 3700 40  0000 C CNN
 F 1 "Sensor_O2_US_narrow" H 7475 3700 40  0000 C CNN
 F 2 "AA_vayu:Sensor_O2_US_narrow" H 7275 3550 40  0001 C CNN
