File: PCB_layout/rtc_ds3231.sch (KiCad schematic (older format))
At the start: 10 parts, among them U2 DS3231N

Commit message: PCB layout, WIP
Parts:
- added BT2: Batt_RTC, AA_vayu:cr2032_03, symbol AA_vayuO2_symbols:Batt_RTC
- BT1: footprint AA_vayu:CR2032 -> AA_vayu:cr2032_02
Connections:
- net BAT: now also BT2.1 (+)
- net GND: now also BT2.2 (-)
Other:
- note added: "Extra footprint for\nalternate battery holder"
Changed lines of the file:
@@
 F 0 "BT1" V 1900 3125 40  0000 C CNN
 F 1 "Batt_RTC" H 2150 3125 40  0000 C CNN
-F 2 "AA_vayu:CR2032" H 2000 3200 60  0001 C CNN
+F 2 "AA_vayu:cr2032_02" H 2000 3200 60  0001 C CNN
 F 3 "" H 2000 3200 60  0000 C CNN
 F 4 "BU2032SM-HD-GCT-ND " H 2100 3500 60  0001 C CNN "Digikey"
@@
 Text Notes 3400 4575 0    60   ~ 12
 DS3231SN#T&R\nSOIC 16, 300 mil
+$Comp
+L AA_vayuO2_symbols:Batt_RTC BT2
+U 1 1 615CBA5D
+P 1675 3200
+F 0 "BT2" V 1575 3125 40  0000 C CNN
+F 1 "Batt_RTC" H 1825 3125 40  0000 C CNN
+F 2 "AA_vayu:cr2032_03" H 1675 3200 60  0001 C CNN
+F 3 "" H 1675 3200 60  0000 C CNN
+F 4 "BU2032SM-HD-GCT-ND " H 1775 3500 60  0001 C CNN "Digikey"
+	1    1675 3200
+	0    1    1    0
+$EndComp
+Wire Wire Line
+	1675 2950 1675 2850
+Wire Wire Line
+	1675 2850 2000 2850
+Wire Wire Line
+	1675 3400 1675 3475
+Wire Wire Line
+	1675 3475 2000 3475
+Text Notes 875  3000 0    40   ~ 0
+Extra footprint for\nalternate battery holder
 $EndSCHEMATC

Commit message: BOM, WIP
Parts:
- U2: value DS3231N -> DS3231SN#T&R
Changed lines of the file:
@@
 P 3675 3200
 F 0 "U2" H 3075 3825 50  0000 L CNB
-F 1 "DS3231N" H 3075 3750 50  0000 L CNB
+F 1 "DS3231SN#T&R" H 3350 3200 50  0000 L CNB
 F 2 "AA_vayu:DS3231" H 3675 3200 60  0001 C CNN
 F 3 "~" H 3675 3200 60  0000 C CNN
