File: PCB_layout/vayuO2.kicad_pcb (KiCad board)
At the start: 2 copper layers, 162.6 x 43.8 mm, 82 parts, among them J1 CLK_IN, J17 MISO, J18 3V3, J19 SCK, J2 DAT_IN, J20 SPI, J21 MOSI, J22 RST, J23 GND, J24 qwiic, J25 qwiic, J7 5V, J8 GND, P1 USB_micro, P3 USB-C_breakout, Q1 DDC114TU, U129 ESP-wroom-32, U130 DS3231N, U131 1117-33, U132 CP2102N-A01-GQFN28

Commit message: PCB layout, WIP
Parts:
- removed BITE1, BITE2: Mouse_Bite, ClockIOT_libs:mouse-bite-0.3in-slot_OSH
- removed C27: 100uF/6V3, ClockIOT_libs:c_2917
- removed C28: 1uF/10V, ClockIOT_libs:c_0805
- removed C29, C30, C31: 100nF, ClockIOT_libs:c_0805
- removed HB45, HB46: mtg_hole_3mm_small, ClockIOT_libs:MountingHole_3.2mm_M3
- removed HB47, HB48: mtg_hole_3mm, ClockIOT_libs:MountingHole_3.2mm_M3_Pad_Via
- removed J1: CLK_IN, ClockIOT_libs:1pin
- removed J17: MISO, ClockIOT_libs:BreakOutPad
- removed J18: 3V3, ClockIOT_libs:BreakOutPad
- removed J19: SCK, ClockIOT_libs:BreakOutPad
- removed J2: DAT_IN, ClockIOT_libs:1pin
- removed J20: SPI, ClockIOT_libs:Header_ISP
- removed J21: MOSI, ClockIOT_libs:BreakOutPad
- removed J22: RST, ClockIOT_libs:BreakOutPad
- removed J23: GND, ClockIOT_libs:BreakOutPad
- removed J24, J25: qwiic, ClockIOT_libs:JST_SH_SM04B-SRSS-TB_1x04-1MP_P1.00mm_Horizontal
- removed J8: GND, ClockIOT_libs:1pin
- removed LDR1, LDR2: LDR, ClockIOT_libs:r_0805_ldr_2
- removed P3: USB-C_breakout, ClockIOT_libs:USB-C_bout
- removed S1: SW-ENTER, ClockIOT_libs:SW_SMD_311020004
- removed S2: SW-INC, ClockIOT_libs:SW_SMD_311020004
- removed S3: SW-EN, ClockIOT_libs:SW_SMD_311020004
- removed S6: SW-MODE, ClockIOT_libs:SW_SMD_311020004
- removed U129: ESP-wroom-32, ClockIOT_libs:esp_wroom_32
- removed U130: DS3231N, ClockIOT_libs:DS3231
- removed U131: 1117-33, ClockIOT_libs:SOT-223-3_TabPin2
- removed U132: CP2102N-A01-GQFN28, ClockIOT_libs:QFN-28-1EP_5x5mm_Pitch0.5mm
- added BT2: Batt_RTC, AA_vayu:cr2032_03, F.Cu at (64.6, 114.0)
- added C1: 100uF/6V3, AA_vayu:CP_Elec_10x10, F.Cu at (171.0, 56.0)
- added C10: 100nF, AA_vayu:C_0603_1608Metric, F.Cu at (65.8, 69.2)
- added C11: 100nF, AA_vayu:C_0603_1608Metric, F.Cu at (76.2, 92.2)
- added C12: 10uF/25V, AA_vayu:CP_Elec_6.3x5.4, F.Cu at (80.5, 131.5)
- added C13: 22uF/25V, AA_vayu:CP_Elec_6.3x5.3, F.Cu at (80.5, 124.0)
- added C14: 1nF, AA_vayu:C_0603_1608Metric, F.Cu at (148.8, 124.1)
- added C15: 1nF, AA_vayu:C_0603_1608Metric, F.Cu at (146.1, 122.1)
- added C16: 1nF, AA_vayu:C_0603_1608Metric, F.Cu at (144.5, 119.1)
- added C2: 1uF/10V, AA_vayu:C_0603_1608Metric, F.Cu at (174.7, 62.4)
- added C3: 100nF, AA_vayu:C_0603_1608Metric, F.Cu at (141.3, 76.8)
- added C4: 100nF, AA_vayu:C_0603_1608Metric, F.Cu at (154.3, 76.8)
- added C5: 100nF, AA_vayu:C_0603_1608Metric, F.Cu at (115.0, 108.0)
- added C6: 100nF, AA_vayu:C_0603_1608Metric, F.Cu at (108.4, 108.0)
- added C8: 100nF, AA_vayu:C_0603_1608Metric, F.Cu at (89.0, 118.5)
- added C9: 10uF/25V, AA_vayu:CP_Elec_6.3x5.4, F.Cu at (65.8, 64.2)
- added CN1: Conn_LED, AA_vayu:JST_EH_B3B-EH-A_1x03_P2.50mm_Vertical, F.Cu at (149.0, 53.0)
- added CN10: OUT, AA_vayu:TerminalBlock_Wurth_1377-2_Horizontal, F.Cu at (88.2, 54.8)
- added CN11: OUT, AA_vayu:TerminalBlock_Wurth_1377-2_Horizontal, F.Cu at (98.2, 54.8)
- added CN12: OUT, AA_vayu:TerminalBlock_Wurth_1377-2_Horizontal, F.Cu at (108.2, 54.8)
- added CN13: OUT, AA_vayu:TerminalBlock_Wurth_1377-2_Horizontal, F.Cu at (118.2, 54.8)
- added CN14: Conn_Analog, AA_vayu:JST_EH_B2B-EH-A_1x02_P2.50mm_Vertical, F.Cu at (139.9, 113.4)
- added CN15: Conn_ADS1115, AA_vayu:ADS1115, F.Cu at (135.6, 104.5)
- added CN16: Conn_S1, AA_vayu:JST_EH_B2B-EH-A_1x02_P2.50mm_Vertical, F.Cu at (183.0, 105.0)
- added CN17: Conn_S2, AA_vayu:JST_EH_B2B-EH-A_1x02_P2.50mm_Vertical, F.Cu at (183.0, 100.0)
- added CN18: Conn_S3, AA_vayu:JST_EH_B2B-EH-A_1x02_P2.50mm_Vertical, F.Cu at (183.0, 95.0)
- added CN19: Conn_O2_5V, AA_vayu:JST_EH_B2B-EH-A_1x02_P2.50mm_Vertical, F.Cu at (157.5, 53.0)
- added CN2: UART1, AA_vayu:JST_EH_B4B-EH-A_1x04_P2.50mm_Vertical, F.Cu at (145.2, 75.5)
- added CN3: UART2, AA_vayu:JST_EH_B4B-EH-A_1x04_P2.50mm_Vertical, F.Cu at (150.8, 75.5)
- added CN4: I2C_1, AA_vayu:JST_EH_B4B-EH-A_1x04_P2.50mm_Vertical, F.Cu at (112.0, 106.0)
- added CN5: I2C_2, AA_vayu:JST_EH_B4B-EH-A_1x04_P2.50mm_Vertical, F.Cu at (105.0, 106.0)
- added CN7: 24VDC, AA_vayu:TerminalBlock_Wurth_1377-2_Horizontal, F.Cu at (68.2, 54.8)
- added CN8: USB_micro, AA_vayu:USB_Micro-B_seeed-320010561, F.Cu at (185.3, 119.8)
- added CN9: OUT, AA_vayu:TerminalBlock_Wurth_1377-2_Horizontal, F.Cu at (78.2, 54.8)
- added D10: LED, AA_vayu:LED_0603_1608Metric, F.Cu at (110.8, 80.8)
- added D11: B220A-13-F, AA_vayu:D_SMB, F.Cu at (119.2, 63.0)
- added D12: LED, AA_vayu:LED_0603_1608Metric, F.Cu at (120.8, 80.8)
- added D3: PRTR5V0U2X, AA_vayu:SOT-143, F.Cu at (177.5, 120.1)
- added D4: B220A-13-F, AA_vayu:D_SMB, F.Cu at (79.2, 63.0)
- added D5: LED, AA_vayu:LED_0603_1608Metric, F.Cu at (80.8, 80.8)
- added D6: LED, AA_vayu:LED_0603_1608Metric, F.Cu at (90.8, 80.8)
- added D7: B220A-13-F, AA_vayu:D_SMB, F.Cu at (99.2, 63.0)
- added D8: LED, AA_vayu:LED_0603_1608Metric, F.Cu at (100.8, 80.8)
- added D9: B220A-13-F, AA_vayu:D_SMB, F.Cu at (109.2, 63.0)
- added HB1: mtg_hole_3mm, AA_vayu:MountingHole_3.2mm_M3_Pad_Via, F.Cu at (54.0, 134.0)
- added HB2: mtg_hole_3mm, AA_vayu:MountingHole_3.2mm_M3_Pad_Via, F.Cu at (54.0, 54.0)
- added HB3: mtg_hole_3mm, AA_vayu:MountingHole_3.2mm_M3_Pad_Via, F.Cu at (182.0, 134.0)
- added HB4: mtg_hole_3mm, AA_vayu:MountingHole_3.2mm_M3_Pad_Via, F.Cu at (182.0, 54.0)
- added LS1: Piezo, AA_vayu:JST_EH_B2B-EH-A_1x02_P2.50mm_Vertical, F.Cu at (138.0, 53.0)
- added MB1: Mouse_Bite, AA_vayu:mouse-bite-2.54mm-slot_OSH, F.Cu at (118.0, 179.2)
- added MB2: Mouse_Bite, AA_vayu:mouse-bite-2.54mm-slot_OSH, F.Cu at (227.2, 124.0)
- added MB3: Mouse_Bite, AA_vayu:mouse-bite-2.54mm-slot_OSH, F.Cu at (62.0, 179.2)
- added MB4: Mouse_Bite, AA_vayu:mouse-bite-2.54mm-slot_OSH, F.Cu at (227.2, 94.0)
- added MB5: Mouse_Bite, AA_vayu:mouse-bite-2.54mm-slot_OSH, F.Cu at (174.0, 179.2)
- added MB6: Mouse_Bite, AA_vayu:mouse-bite-2.54mm-slot_OSH, F.Cu at (227.2, 64.0)
- added Q10: BSS138, AA_vayu:SOT-23, F.Cu at (149.6, 66.5)
- added Q11: BSS138, AA_vayu:SOT-23, F.Cu at (149.5, 88.1)
- added Q12: BSS138, AA_vayu:SOT-23, F.Cu at (149.5, 91.7)
- added Q2: DDC114TU, AA_vayu:SOT-363_SC-70-6, F.Cu at (148.8, 117.6)
- added Q3: IRLR7843TRPBF, AA_vayu:MOSFET_D_PAK, F.Cu at (79.2, 72.8)
- added Q4: IRLR7843TRPBF, AA_vayu:MOSFET_D_PAK, F.Cu at (89.2, 72.8)
- added Q5: IRLR7843TRPBF, AA_vayu:MOSFET_D_PAK, F.Cu at (99.2, 72.8)
- added Q6: IRLR7843TRPBF, AA_vayu:MOSFET_D_PAK, F.Cu at (109.2, 72.8)
- added Q7: IRLR7843TRPBF, AA_vayu:MOSFET_D_PAK, F.Cu at (119.2, 72.8)
- added Q8: BSS138, AA_vayu:SOT-23, F.Cu at (146.8, 58.5)
- added Q9: BSS138, AA_vayu:SOT-23, F.Cu at (149.6, 70.2)
- added R1: 10k, AA_vayu:R_0603_1608Metric, F.Cu at (176.0, 105.0)
- added R15: 1k, AA_vayu:R_0603_1608Metric, F.Cu at (160.5, 113.1)
- added R17: 470E, AA_vayu:R_0603_1608Metric, F.Cu at (148.8, 115.1)
- added R2: 10k, AA_vayu:R_0603_1608Metric, F.Cu at (176.0, 100.0)
- added R26: 1k, AA_vayu:R_0603_1608Metric, F.Cu at (87.2, 82.8)
- added R27: 10k, AA_vayu:R_0603_1608Metric, F.Cu at (90.8, 82.8)
- added R28: 470E, AA_vayu:R_0603_1608Metric, F.Cu at (101.2, 96.2)
- added R29: 100E, AA_vayu:R_0603_1608Metric, F.Cu at (97.2, 80.8)
- added R30: 1k, AA_vayu:R_0603_1608Metric, F.Cu at (97.2, 82.8)
- added R31: 10k, AA_vayu:R_0603_1608Metric, F.Cu at (100.8, 82.8)
- added R32: 470E, AA_vayu:R_0603_1608Metric, F.Cu at (104.2, 96.2)
- added R33: 100E, AA_vayu:R_0603_1608Metric, F.Cu at (107.2, 80.8)
- added R34: 1k, AA_vayu:R_0603_1608Metric, F.Cu at (107.2, 82.8)
- added R35: 10k, AA_vayu:R_0603_1608Metric, F.Cu at (110.8, 82.8)
- added R36: 470E, AA_vayu:R_0603_1608Metric, F.Cu at (107.2, 96.2)
- added R37: 100E, AA_vayu:R_0603_1608Metric, F.Cu at (117.2, 80.8)
- added R38: 1k, AA_vayu:R_0603_1608Metric, F.Cu at (117.2, 82.8)
- added R39: 10k, AA_vayu:R_0603_1608Metric, F.Cu at (120.8, 82.8)
- added R40: 10k, AA_vayu:R_0603_1608Metric, F.Cu at (149.5, 58.2)
- added R41: 10k, AA_vayu:R_0603_1608Metric, F.Cu at (144.0, 58.2)
- added R42: 10k, AA_vayu:R_0603_1608Metric, F.Cu at (153.0, 71.2)
- added R43: 10k, AA_vayu:R_0603_1608Metric, F.Cu at (146.2, 71.2)
- added R44: 10k, AA_vayu:R_0603_1608Metric, F.Cu at (153.0, 67.5)
- added R45: 10k, AA_vayu:R_0603_1608Metric, F.Cu at (146.2, 67.5)
- added R46: 10k, AA_vayu:R_0603_1608Metric, F.Cu at (152.9, 89.1)
- added R47: 10k, AA_vayu:R_0603_1608Metric, F.Cu at (146.1, 89.1)
- added R48: 10k, AA_vayu:R_0603_1608Metric, F.Cu at (152.9, 92.7)
- added R49: 10k, AA_vayu:R_0603_1608Metric, F.Cu at (146.1, 92.7)
- added R50: 1k, AA_vayu:R_0603_1608Metric, F.Cu at (136.3, 56.7)
- added R51: 0E, AA_vayu:SolderJumper-2_P1.3mm_Open_RoundedPad1.0x1.5mm, B.Cu at (130.1, 115.9)
- added R52: 0E, AA_vayu:SolderJumper-2_P1.3mm_Open_RoundedPad1.0x1.5mm, B.Cu at (130.1, 113.4)
- added R53: 0E, AA_vayu:SolderJumper-2_P1.3mm_Open_RoundedPad1.0x1.5mm, B.Cu at (130.1, 110.8)
- added R54: 0E, AA_vayu:SolderJumper-2_P1.3mm_Open_RoundedPad1.0x1.5mm, B.Cu at (130.1, 108.3)
- added R55: 0E, AA_vayu:SolderJumper-2_P1.3mm_Open_RoundedPad1.0x1.5mm, B.Cu at (139.9, 100.7)
- added R56: 0E, AA_vayu:SolderJumper-2_P1.3mm_Open_RoundedPad1.0x1.5mm, B.Cu at (139.9, 98.2)
- added R57: 0E, AA_vayu:SolderJumper-2_P1.3mm_Open_RoundedPad1.0x1.5mm, B.Cu at (139.9, 95.6)
- added R58: 0E, AA_vayu:SolderJumper-2_P1.3mm_Open_RoundedPad1.0x1.5mm, B.Cu at (139.9, 93.1)
- added U1: ESP32-WROOM-32UC, AA_vayu:ESP_wroom_32_ext_ant, F.Cu at (160.3, 77.2)
- added U10: Sensor_O2_US_narrow, AA_vayu:Sensor_O2_US_narrow, F.Cu at (240.0, 94.0)
- added U11: DC_DC_buck_6W, AA_vayu:DC_DC_conv_6W, F.Cu at (72.5, 78.2)
- added U2: DS3231N, AA_vayu:DS3231, F.Cu at (88.0, 111.5)
- added U3: B2405S-2WR2, AA_vayu:DC_DC_conv_2W, F.Cu at (67.5, 78.2)
- added U4: LM1117-33, AA_vayu:TO-252-3_TabPin2, F.Cu at (92.0, 127.8)
- added U5: CP2102N-A01-GQFN28, AA_vayu:QFN-28-1EP_5x5mm_Pitch0.5mm, F.Cu at (155.6, 112.1)
- added U6: 24V_BUCK, AA_vayu:DC_DC_buck_LM2596_Vertical, F.Cu at (57.8, 80.8)
- added U7: Sensor_O2_US, AA_vayu:Sensor_O2_US, F.Cu at (118.0, 192.0)
- added U8: PS2801-4, AA_vayu:SO-16_5.3x10.2mm_P1.27mm, F.Cu at (100.2, 89.5)
- added U9: PS2801-4, AA_vayu:SO-4_5.3x2.7mm_P1.27mm, F.Cu at (107.2, 89.5)
- BT1: footprint ClockIOT_libs:CR2032_SMD_SKST-2007D -> AA_vayu:cr2032_02
- C17: footprint ClockIOT_libs:c_2917 -> AA_vayu:CP_Elec_6.3x5.4
- C18: value 22uF/25V -> 100nF; footprint ClockIOT_libs:c_2917 -> AA_vayu:C_0603_1608Metric
- C19: value 1nF -> 10uF/25V; footprint ClockIOT_libs:c_0805 -> AA_vayu:CP_Elec_6.3x5.4
- C20, C21: value 1nF -> 100nF; footprint ClockIOT_libs:c_0805 -> AA_vayu:C_0603_1608Metric
- C22, C24, C26: footprint ClockIOT_libs:c_0805 -> AA_vayu:C_0603_1608Metric
- C23, C25: value 10uF/25V -> 100nF; footprint ClockIOT_libs:c_2917 -> AA_vayu:C_0603_1608Metric
- D1: value PRTR5V0U2X -> B220A-13-F; footprint ClockIOT_libs:SOT-143 -> AA_vayu:D_SMB
- D2: footprint ClockIOT_libs:LED-0805 -> AA_vayu:LED_0603_1608Metric
- G1: footprint ClockIOT_libs:Logo-WL3 -> AA_vayu:logo_butterfly_silk_15x12
- G2: footprint ClockIOT_libs:KiCad-Logo2_6mm_SilkScreen -> AA_vayu:KiCad-Logo2_6mm_SilkScreen
- G3: footprint ClockIOT_libs:OSHW_6mm -> AA_vayu:Logo_silk_OSHW_6x6mm
- J7: value 5V -> Conn_01x01; footprint ClockIOT_libs:1pin -> AA_vayu:BreakOutPad
- JP1: footprint ClockIOT_libs:R_0402 -> AA_vayu:R_0402
- L1, L2, R3, R6, R8: footprint ClockIOT_libs:r_0805 -> AA_vayu:R_0603_1608Metric
- P1: value USB_micro -> USB-C_breakout; footprint ClockIOT_libs:USB_Micro-B_seeed-320010561 -> AA_vayu:USB-C_bout
- Q1: value DDC114TU -> MMBT3904; footprint ClockIOT_libs:SOT-363_SC-70-6 -> AA_vayu:SOT-23
- R10, R12, R24: value 10k -> 470E; footprint ClockIOT_libs:r_0805 -> AA_vayu:R_0603_1608Metric
- R11: value 10k -> 1k; footprint ClockIOT_libs:r_0805 -> AA_vayu:R_0603_1608Metric
- R13, R14: value 10k -> 0E NC; footprint ClockIOT_libs:r_0805 -> AA_vayu:R_0603_1608Metric
- R16, R18: value 470R -> 0E; footprint ClockIOT_libs:r_0805 -> AA_vayu:R_0603_1608Metric
- R19: value 0R NC -> 10k; footprint ClockIOT_libs:r_0805 -> AA_vayu:R_0603_1608Metric
- R20: value 0R NC -> 470E; footprint ClockIOT_libs:r_0805 -> AA_vayu:R_0603_1608Metric
- R21: value 0R -> 100E; footprint ClockIOT_libs:r_0805 -> AA_vayu:R_0603_1608Metric
- R22: value 470R -> 1k; footprint ClockIOT_libs:r_0805 -> AA_vayu:R_0603_1608Metric
- R23: value 0R -> 10k; footprint ClockIOT_libs:r_0805 -> AA_vayu:R_0603_1608Metric
- R25: value 10k -> 100E; footprint ClockIOT_libs:r_0805 -> AA_vayu:R_0603_1608Metric
- R4: value 1k -> 220E; footprint ClockIOT_libs:r_0805 -> AA_vayu:R_0603_1608Metric
- R5: value 1k -> 10k; footprint ClockIOT_libs:r_0805 -> AA_vayu:R_0603_1608Metric
- R7: value 10k -> 4K7; footprint ClockIOT_libs:r_0805 -> AA_vayu:R_0603_1608Metric
- R9: value 4K7 -> 10k; footprint ClockIOT_libs:r_0805 -> AA_vayu:R_0603_1608Metric
- S4: value SW-BOOT -> SW-EN; footprint ClockIOT_libs:SW_SMD_311020004 -> AA_vayu:SW_SMD_311020004; moved to F.Cu
- S5: value SW-DEC -> SW-BOOT; footprint ClockIOT_libs:SW_SMD_311020004 -> AA_vayu:SW_SMD_311020004; moved to F.Cu
- TP1: value ~RST -> SQR; footprint ClockIOT_libs:BreakOutPad -> AA_vayu:BreakOutPad; moved to F.Cu
- TP2: value SQR -> ~RST; footprint ClockIOT_libs:BreakOutPad -> AA_vayu:BreakOutPad; moved to F.Cu
- TP3: footprint ClockIOT_libs:BreakOutPad -> AA_vayu:BreakOutPad; moved to F.Cu
- moved BT1 141.2 mm to (66.1, 114.0), turned to 90 degrees
- moved G3 140.2 mm to (113.5, 192.8), turned to 0 degrees
- moved P1 140.0 mm to (183.4, 119.7)
- moved G2 134.9 mm to (100.5, 186.2), turned to 0 degrees
- moved L1 133.0 mm to (180.3, 125.6), turned to 0 degrees
- moved L2 127.2 mm to (180.3, 113.8), turned to 0 degrees
- moved C20 120.7 mm to (160.6, 115.1)
- moved TP2 112.2 mm to (95.5, 108.3)
- moved TP3 112.1 mm to (95.5, 103.2)
- moved TP1 108.7 mm to (95.5, 105.8)
- moved G1 106.9 mm to (93.0, 190.0), turned to 0 degrees
- moved R16 106.8 mm to (148.9, 113.1), turned to 0 degrees
- moved R7 100.8 mm to (94.5, 118.4), turned to 180 degrees
- moved R6 99.2 mm to (92.5, 103.8), turned to 270 degrees
- moved S5 95.0 mm to (155.0, 132.0), turned to 90 degrees
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Connections:
- C17 pad 1: /5V -> /3V3
- C19 pad 1: /EN -> /5V
- C20 pad 1: Net-(C20-Pad1) -> /5V
- C21 pad 1: GND -> /mosfets/filter1
- C21 pad 2: Net-(C21-Pad2) -> GND
- C22 pad 1: /rtc_ds3231/BAT -> /mosfets/filter2
- C23 pad 1: /3V3 -> /mosfets/filter3
- C24 pad 1: /3V3 -> /mosfets/filter4
- C25 pad 1: /5V -> /mosfets/filter5
- C26 pad 1: /5V -> GND
- C26 pad 2: GND -> Net-(C26-Pad2)
- D1 pad 1: GND -> +24V
- D1 pad 2: /esp_pwr_uart/USB_D- -> /mosfets/OP2
- J7 pad 1: /5V -> /ALRT
- L2 pad 2: Net-(L2-Pad2) -> Net-(CN8-Pad6)
- P1 pad 2: /esp_pwr_uart/USB_D- -> /esp_pwr_uart/VBUS
- P1 pad 3: /esp_pwr_uart/USB_D+ -> /esp_pwr_uart/USB_D-
- P1 pad 4: Net-(P1-Pad4) -> /esp_pwr_uart/USB_D+
- P1 pad 5: GND -> Net-(P1-Pad5)
- P1 pad 6: Net-(L2-Pad2) -> Net-(P1-Pad6)
- Q1 pad 1: /esp_pwr_uart/RTS -> Net-(C26-Pad2)
- Q1 pad 2: /DTR -> GND
- Q1 pad 3: /IO0 -> Net-(LS1-Pad1)
- R10 pad 1: /SW_E -> Net-(C15-Pad1)
- R10 pad 2: GND -> /EN
- R11 pad 1: /SW_I -> Net-(D2-Pad1)
- R11 pad 2: GND -> /5V
- R12 pad 1: GND -> Net-(C16-Pad2)
- R12 pad 2: /LDR1 -> /IO0
- R13 pad 1: /LDR2 -> /IO15
- R13 pad 2: GND -> /esp_pwr_uart/CTS
- R14 pad 1: /esp_pwr_uart/ACTIVE -> /IO13
- R14 pad 2: GND -> /esp_pwr_uart/RTS
- R16 pad 1: Net-(C20-Pad1) -> /TXD0
- R16 pad 2: /EN -> /esp_pwr_uart/RXD
- R18 pad 1: Net-(C21-Pad2) -> /RXD0
- R18 pad 2: /IO0 -> /esp_pwr_uart/TXD
- R19 pad 1: /IO15 -> /esp_pwr_uart/ACTIVE
- R19 pad 2: /esp_pwr_uart/CTS -> GND
- R20 pad 1: /IO13 -> /OUT1
- R20 pad 2: /esp_pwr_uart/RTS -> /mosfets/filter1
- R21 pad 1: /TXD0 -> Net-(Q3-Pad1)
- R21 pad 2: /esp_pwr_uart/RXD -> Net-(R21-Pad2)
- R22 pad 2: /esp_pwr_uart/TXD -> Net-(R21-Pad2)
- R23 pad 1: /RXD0 -> GNDPWR
- R23 pad 2: /esp_pwr_uart/TXD -> Net-(R21-Pad2)
- R24 pad 1: /SW_D -> /OUT2
- R24 pad 2: GND -> /mosfets/filter2
- R25 pad 1: /SW_M -> Net-(Q4-Pad1)
- R25 pad 2: GND -> Net-(R25-Pad2)
- R3 pad 1: /3V3 -> /SW_M
- R3 pad 2: /EN -> GND
- R4 pad 1: Net-(D2-Pad1) -> Net-(C26-Pad2)
- R4 pad 2: /5V -> /SPKR
- R5 pad 2: /esp_pwr_uart/RSTb -> /rtc_ds3231/SQR
- R6 pad 2: /rtc_ds3231/SQR -> /rtc_ds3231/32kHz
- R7 pad 2: /rtc_ds3231/32kHz -> /SCL
- R8 pad 2: /SCL -> /SDA
- R9 pad 2: /SDA -> /EN
- S4 pad 2: Net-(C21-Pad2) -> Net-(C15-Pad1)
- S4 pad 4: Net-(C21-Pad2) -> Net-(C15-Pad1)
- S5 pad 1: /3V3 -> GND
- S5 pad 2: /SW_D -> Net-(C16-Pad2)
- S5 pad 3: /3V3 -> GND
- S5 pad 4: /SW_D -> Net-(C16-Pad2)
- TP1 pad 1: /rtc_ds3231/RESET -> /rtc_ds3231/SQR
- TP2 pad 1: /rtc_ds3231/SQR -> /rtc_ds3231/RESET
Routing:
- net GND: track 793.3 -> 401.2 mm, vias 57 -> 36
- net /5V: track 150.6 -> 434.9 mm, vias 0 -> 6
- net GNDPWR: track 0.00 -> 221.7 mm, vias 0 -> 15
- net +24V: track 0.00 -> 169.2 mm
- net /EN: track 130.3 -> 10.1 mm, vias 3 -> 0
- net /SW_M: track 128.9 -> 23.1 mm, vias 1 -> 0
- net /OUT1: track 0.00 -> 98.0 mm
- net /OUT2: track 0.00 -> 96.2 mm
- net /CLK_IN: track 94.9 -> 0.00 mm, vias 1 -> 0
- net /OUT3: track 0.00 -> 94.3 mm
- net /OUT4: track 0.00 -> 92.5 mm
- net /OUT5: track 0.00 -> 91.0 mm
- net /SW_D: track 113.6 -> 28.6 mm, vias 1 -> 0
- net /DAT_IN: track 81.9 -> 0.00 mm, vias 1 -> 0
- net /SW_E: track 79.0 -> 0.00 mm, vias 1 -> 0
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- added copper zone on B.Cu, net /mosfets/OP1
- added copper zone on F.Cu, net /mosfets/OP1
- added copper zone on B.Cu, net /mosfets/OP2
- added copper zone on F.Cu, net /mosfets/OP2
- added copper zone on B.Cu, net /mosfets/OP3
- added copper zone on F.Cu, net /mosfets/OP3
- added copper zone on B.Cu, net /mosfets/OP4
- added copper zone on F.Cu, net /mosfets/OP4
- added copper zone on B.Cu, net /mosfets/OP5
- added copper zone on F.Cu, net /mosfets/OP5
- removed copper zone on F.Cu, net /5V
- removed copper zone on F.Cu, net Net-(C21-Pad2)
Other:
- board size 162.6 x 43.8 mm -> 201.5 x 153.5 mm
- net class 0.25mm added: clearance 0.1016, trace_width 0.25, via_dia 0.9, via_drill 0.5
- net class 0.2mm added: clearance 0.1016, trace_width 0.2, via_dia 0.9, via_drill 0.5
- net class 0.5mm added: clearance 0.1016, trace_width 0.5, via_dia 0.9, via_drill 0.5
- net class 1.0mm added: clearance 0.1016, trace_width 1, via_dia 0.9, via_drill 0.5
- net class 2.0mm added: clearance 0.1016, trace_width 2, via_dia 0.9, via_drill 0.5
- net class 20mil removed
- net class 30mil removed
- net class 40mil removed
- net class 8 mil removed
- net class Power removed
- board text removed: "3V3"
- board text removed: "3V3 MOSI GND"
- board text removed: "5V"
- board text removed: "BOOT"
- board text removed: "CC1"
- board text removed: "CC2"
- board text removed: "CLK"
- board text removed: "CLK_IN"
- board text removed: "CMD"
- board text removed: "CONTROLLER"
- board text removed: "ClockIOT"
- board text removed: "D+"
- board text removed: "D-"
- board text removed: "DAT_IN"
- board text removed: "DEC"
- board text removed: "EN"
- board text removed: "ENTER"
- board text removed: "GND"
- board text removed: "GND|3V3|SDA|SCL"
- board text removed: "INC"
- board text removed: "IO0"
- board text removed: "IO12"
- board text removed: "IO13"
- board text removed: "IO14"
- board text removed: "IO15"
- board text removed: "IO2"
- board text removed: "IO21/SDA"
- board text removed: "IO22/SCL"
- board text removed: "IO23"
- board text removed: "IO25"
- board text removed: "IO26"
- board text removed: "IO27"
- board text removed: "IO34"
- board text removed: "IO35"
- board text removed: "LDR1"
- board text removed: "LDR2"
- board text removed: "MISO SCK RST"
- board text removed: "MODE"
- board text removed: "NC"
- board text removed: "RXD0"
- board text removed: "SBU1"
- board text removed: "SBU2"
- board text removed: "SD2"
- board text removed: "SD3"
- board text removed: "SDI"
- board text removed: "SDO"
- board text removed: "SENSOR_VN"
- board text removed: "SENSOR_VP"
- board text removed: "SW_D"
- board text removed: "SW_E"
- board text removed: "SW_I"
- board text removed: "SW_M"
- board text removed: "TXD0"
- board text removed: "VBUS"
- board text removed: "github.com/wyolum/ClockIOT"
- board text removed: "hardware"
- board text removed: "open source"
- board text removed: "rev 5"
- board text removed: "wyolum.com"

Commit message: BOM, WIP
Parts:
- removed MB1, MB2, MB3, MB4, MB5, MB6: Mouse_Bite, AA_vayu:mouse-bite-2.54mm-slot_OSH
- removed U10: Sensor_O2_US_narrow, AA_vayu:Sensor_O2_US_narrow
- removed U7: Sensor_O2_US, AA_vayu:Sensor_O2_US
- C1: footprint AA_vayu:CP_Elec_10x10 -> AA_vayu:CP_Elec_8x10
- C12, C17, C9: footprint AA_vayu:CP_Elec_6.3x5.4 -> AA_vayu:CP_Elec_6.3x7.7
- C13: footprint AA_vayu:CP_Elec_6.3x5.3 -> AA_vayu:CP_Elec_6.3x7.7
- G1, G2, G3: moved to B.Cu
- Q2: value DDC114TU -> DTC123YCA
- U2: value DS3231N -> DS3231SN#T&R
- U9: value PS2801-4 -> PS2801-1
- moved G3 63.8 mm to (94.4, 131.9), turned to 180 degrees
- moved G1 62.8 mm to (106.2, 128.6), turned to 180 degrees
- moved G2 56.4 mm to (84.7, 132.1), turned to 180 degrees
- moved CN5 40.9 mm to (145.2, 98.5)
- moved C5 40.1 mm to (154.3, 99.8)
- moved CN4 39.5 mm to (150.8, 98.5)
- moved S4 37.5 mm to (128.5, 132.0)
- moved S5 37.0 mm to (118.0, 132.0)
- moved C6 33.9 mm to (141.3, 99.8)
- moved C17 27.9 mm to (143.8, 124.8), turned to 180 degrees
- moved C19 27.1 mm to (143.8, 132.0), turned to 180 degrees
- moved C16 24.3 mm to (166.8, 128.8), turned to 90 degrees
- moved C15 24.3 mm to (170.3, 122.3), turned to 90 degrees
- moved R12 23.6 mm to (165.0, 128.8), turned to 90 degrees
- moved R19 19.8 mm to (156.4, 130.5), turned to 270 degrees
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Routing:
- net GND: track 401.2 -> 890.4 mm, vias 36 -> 37
- net /3V3: track 378.0 -> 555.8 mm, vias 12 -> 4
- net /EN: track 10.1 -> 98.9 mm, vias 0 -> 3
- net /RXD0: track 3.00 -> 56.1 mm, vias 0 -> 3
- net /IO13: track 2.99 -> 56.0 mm, vias 0 -> 4
- net /IO0: track 8.29 -> 53.3 mm, vias 0 -> 1
- net /TXD0: track 3.00 -> 48.0 mm, vias 0 -> 1
- net Net-(C16-Pad2): track 26.1 -> 70.9 mm
- net /IO15: track 2.99 -> 44.2 mm, vias 0 -> 2
- net Net-(C15-Pad1): track 36.1 -> 65.3 mm
- net /5V: track 434.9 -> 457.8 mm, vias 6 -> 8
- net GNDPWR: track 221.7 -> 242.5 mm
- net /esp_pwr_uart/RTS: track 5.80 -> 22.5 mm, vias 0 -> 2
- net /rtc_ds3231/RESET: track 22.1 -> 5.84 mm
- net /esp_pwr_uart/USB_D+: track 39.0 -> 55.1 mm, vias 2 -> 1
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Other:
- board size 201.5 x 153.5 mm -> 136 x 88 mm
- net class 0.2mm removed
- net class 1.5mm added: clearance 0.1016, trace_width 1.5, via_dia 0.9, via_drill 0.5
- net class 10mil removed
- net class 2.0mm removed
- rule trace_min: 0.08 -> 0

Commit message: final production files generated
Parts:
- added U12: PS2801-1, AA_vayu:SO-4_5.3x2.7mm_P1.27mm, F.Cu at (101.5, 89.5)
- added U7: PS2801-1, AA_vayu:SO-4_5.3x2.7mm_P1.27mm, F.Cu at (95.1, 89.5)
- added U9: PS2801-1, AA_vayu:SO-4_5.3x2.7mm_P1.27mm, F.Cu at (98.3, 89.5)
- added kibuzzard-615EFBF6: G***, AA_vayu:label_wyolum, B.Cu at (103.9, 127.1)
- added kibuzzard-615EFE42: G***, AA_vayu:label_24V, F.Cu at (65.7, 58.6)
- added kibuzzard-615EFE7C: G***, label, F.Cu at (75.8, 58.4)
- added kibuzzard-615EFF0D: G***, AA_vayu:label_out2, F.Cu at (85.7, 58.4)
- added kibuzzard-615EFF16: G***, AA_vayu:label_out3, F.Cu at (95.8, 58.4)
- added kibuzzard-615EFF1D: G***, AA_vayu:label_out4, F.Cu at (105.7, 58.4)
- added kibuzzard-615EFF24: G***, AA_vayu:label_out5, F.Cu at (115.8, 58.4)
- added kibuzzard-615F0132: G***, AA_vayu:label_boot, F.Cu at (118.0, 127.4)
- added kibuzzard-615F016F: G***, label, F.Cu at (128.5, 127.4)
- added kibuzzard-615F01C3: G***, AA_vayu:label_ads1115, F.Cu at (124.8, 93.6)
- added kibuzzard-615F0246: G***, AA_vayu:label_pm, F.Cu at (139.6, 99.7)
- added kibuzzard-615F02BE: G***, AA_vayu:label_I2C_1, F.Cu at (155.0, 107.5)
- added kibuzzard-615F0326: G***, AA_vayu:label_I2C_2, F.Cu at (140.4, 107.5)
- added kibuzzard-615F03BD: G***, AA_vayu:label_uart1, F.Cu at (140.4, 84.6)
- added kibuzzard-615F0408: G***, AA_vayu:label_uart2, F.Cu at (155.1, 84.5)
- added kibuzzard-615F0476: G***, AA_vayu:label_buz, F.Cu at (136.8, 55.7)
- added kibuzzard-615F04CC: G***, AA_vayu:label_O2, F.Cu at (156.2, 55.7)
- added kibuzzard-615F0547: G***, AA_vayu:label_LED, F.Cu at (146.5, 55.7)
- added kibuzzard-615F0858: G***, AA_vayu:label_sw_m, F.Cu at (175.0, 93.8)
- added kibuzzard-615F0877: G***, AA_vayu:label_sw_d, F.Cu at (175.0, 98.8)
- added kibuzzard-615F08E2: G***, AA_vayu:label_sw_i, F.Cu at (175.0, 103.8)
- added kibuzzard-615F0BBC: G***, AA_vayu:label_vayu, F.Cu at (104.7, 110.1)
- added kibuzzard-615F0C20: G***, AA_vayu:label_rev, F.Cu at (104.7, 113.5)
- C19: footprint AA_vayu:CP_Elec_6.3x5.4 -> AA_vayu:CP_Elec_6.3x7.7
- U8: value PS2801-4 -> PS2801-1; footprint AA_vayu:SO-16_5.3x10.2mm_P1.27mm -> AA_vayu:SO-4_5.3x2.7mm_P1.27mm
- moved G2 16.7 mm to (101.4, 132.1)
- moved G3 16.7 mm to (111.1, 131.9)
- moved G1 11.0 mm to (106.2, 117.6)
- moved U8 4.40 mm to (104.7, 89.5)
- moved R1 1.70 mm to (176.0, 106.7)
- moved R2 1.70 mm to (176.0, 101.7)
- moved R3 1.70 mm to (176.0, 96.7)
- moved R20 1.00 mm to (94.3, 96.3)
- moved C21 0.90 mm to (95.9, 96.3)
- moved R24 0.80 mm to (97.5, 96.3)
- moved C22 0.70 mm to (99.1, 96.3)
- moved U10 0.60 mm to (107.9, 89.5)
- moved R28 0.60 mm to (100.7, 96.3)
- moved C23 0.50 mm to (102.3, 96.3)
- moved R32 0.40 mm to (103.9, 96.3)
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- renumbered U9 to U10
Connections:
- U8 pad 1: /mosfets/filter1 -> /mosfets/filter4
- U8 pad 3: /mosfets/filter2 -> GNDPWR
- U8 pad 4: GND -> Net-(R33-Pad2)
Routing:
- net GNDPWR: track 242.5 -> 286.1 mm
- net GND: track 890.4 -> 888.5 mm, vias 37 -> 38
- net /OUT1: track 98.2 -> 99.6 mm
- net Net-(R21-Pad2): track 25.8 -> 24.5 mm
- net /OUT2: track 96.3 -> 97.5 mm
- net /SW_M: track 21.8 -> 22.9 mm
- net /SW_D: track 27.3 -> 28.5 mm
- net /SW_I: track 32.8 -> 33.9 mm
- net Net-(R33-Pad2): track 12.4 -> 11.3 mm
- net /OUT3: track 94.5 -> 95.5 mm
- net Net-(R25-Pad2): track 18.7 -> 17.7 mm
- net /OUT4: track 92.7 -> 93.5 mm
- net Net-(R37-Pad2): track 19.6 -> 18.9 mm
- net /OUT5: track 91.0 -> 91.6 mm
Other:
- outline, holes or cut-outs redrawn
