File: PCB_layout_v2/vayuO2.kicad_pcb (KiCad board)
At the start: 2 copper layers, 124 x 88 mm, 166 parts, among them CN1 Conn_LED, CN10 OUT, CN11 OUT, CN12 OUT, CN13 OUT, CN14 Conn_Analog, CN15 Conn_ADS1115, CN16 Conn_S1, CN17 Conn_S2, CN18 Conn_S3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

Commit message: version 2 ready - production files generated
Parts:
- removed kibuzzard-615F0C20: #G***, AA_vayu:label_rev
- added kibuzzard-6163C896: G***, AA_vayu:label_rev2, F.Cu at (123.0, 136.5)
Routing:
- net /3V3: track 474.9 -> 441.7 mm, vias 49 -> 52
- net GND: track 108.0 -> 104.8 mm
