File: PCB_layout_v3/mosfets.sch (KiCad schematic (older format))
At the start: 50 parts, among them CN10 OUT, CN11 OUT, CN12 OUT, CN13 OUT, CN9 OUT, Q3 IRF540NS, Q4 IRF540NS, Q5 IRF540NS, Q6 IRF540NS, Q7 IRF540NS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

Commit message: Updated component footprint
* Updated opto IC footprint

Co-Authored-By: Anool Mahidharia <anool.m@gmail.com>
Parts:
- U5: renamed from U7; value PS2801-1 -> PS2801-4; footprint AA_vayu:SO-4_5.3x2.7mm_P1.27mm -> AA_vayu:SO-16_5.3x10.2mm_P1.27mm; symbol AA_vayuO2_symbols:PS2801-1 -> AA_vayuO2_symbols:PS2801-4
- U5: renamed from U9; value PS2801-1 -> PS2801-4; footprint AA_vayu:SO-4_5.3x2.7mm_P1.27mm -> AA_vayu:SO-16_5.3x10.2mm_P1.27mm; symbol AA_vayuO2_symbols:PS2801-1 -> AA_vayuO2_symbols:PS2801-4
- U5: renamed from U12; value PS2801-1 -> PS2801-4; footprint AA_vayu:SO-4_5.3x2.7mm_P1.27mm -> AA_vayu:SO-16_5.3x10.2mm_P1.27mm; symbol AA_vayuO2_symbols:PS2801-1 -> AA_vayuO2_symbols:PS2801-4
- U5: renamed from U8; value PS2801-1 -> PS2801-4; footprint AA_vayu:SO-4_5.3x2.7mm_P1.27mm -> AA_vayu:SO-16_5.3x10.2mm_P1.27mm; symbol AA_vayuO2_symbols:PS2801-1 -> AA_vayuO2_symbols:PS2801-4
Connections:
- net GND: now also U5.4 (K), U5.6 (K), U5.8 (K); no longer U5.2 (K), U5.2 (K), U5.2 (K)
- net GNDPWR: now also U5.11 (K), U5.13 (E), U5.15 (E), U5.9 (E); no longer U5.3 (E), U5.3 (E), U5.3 (E), U5.3 (E)
- net filter2: now also U5.3 (A); no longer U5.1 (A)
- net filter3: now also U5.5 (A); no longer U5.1 (A)
- net filter4: now also U5.7 (A); no longer U5.1 (A)
- net at R21.2, R22.2, R23.2: now also U5.16 (C); no longer U5.4 (C)
- net at R25.2, R26.2, R27.2: now also U5.14 (C); no longer U5.4 (C)
- net at R29.2, R30.2, R31.2: now also U5.12 (C); no longer U5.4 (C)
- net at R33.2, R34.2, R35.2: now also U5.10 (C); no longer U5.4 (C)
Changed lines of the file:
@@
 	4025 1025 4025 925
 $Comp
-L AA_vayuO2_symbols:PS2801-1 U7
+L AA_vayuO2_symbols:PS2801-4 U5
 U 1 1 616348AD
 P 2325 1425
-F 0 "U7" H 2350 1725 50  0000 C CNN
-F 1 "PS2801-1" H 2350 1625 40  0000 C CNN
-F 2 "AA_vayu:SO-4_5.3x2.7mm_P1.27mm" H 2325 1125 50  0001 C CIN
+F 0 "U5" H 2350 1725 50  0000 C CNN
+F 1 "PS2801-4" H 2350 1625 40  0000 C CNN
+F 2 "AA_vayu:SO-16_5.3x10.2mm_P1.27mm" H 2325 1125 50  0001 C CIN
 F 3 "" H 2300 1400 50  0001 L CNN
 	1    2325 1425
@@
 	4025 2725 4025 2625
 $Comp
-L AA_vayuO2_symbols:PS2801-1 U9
-U 1 1 61650FE4
+L AA_vayuO2_symbols:PS2801-4 U5
+U 2 1 61650FE4
 P 2325 3125
-F 0 "U9" H 2350 3425 50  0000 C CNN
-F 1 "PS2801-1" H 2350 3325 40  0000 C CNN
-F 2 "AA_vayu:SO-4_5.3x2.7mm_P1.27mm" H 2325 2825 50  0001 C CIN
+F 0 "U5" H 2350 3425 50  0000 C CNN
+F 1 "PS2801-4" H 2350 3325 40  0000 C CNN
+F 2 "AA_vayu:SO-16_5.3x10.2mm_P1.27mm" H 2325 2825 50  0001 C CIN
 F 3 "" H 2300 3100 50  0001 L CNN
-	1    2325 3125
+	2    2325 3125
 	1    0    0    -1
 $EndComp
@@
 	4025 4425 4025 4325
 $Comp
-L AA_vayuO2_symbols:PS2801-1 U12
-U 1 1 6165FC0E
+L AA_vayuO2_symbols:PS2801-4 U5
+U 3 1 6165FC0E
 P 2325 4825
-F 0 "U12" H 2350 5125 50  0000 C CNN
-F 1 "PS2801-1" H 2350 5025 40  0000 C CNN
-F 2 "AA_vayu:SO-4_5.3x2.7mm_P1.27mm" H 2325 4525 50  0001 C CIN
+F 0 "U5" H 2350 5125 50  0000 C CNN
+F 1 "PS2801-4" H 2350 5025 40  0000 C CNN
+F 2 "AA_vayu:SO-16_5.3x10.2mm_P1.27mm" H 2325 4525 50  0001 C CIN
 F 3 "" H 2300 4800 50  0001 L CNN
-	1    2325 4825
+	3    2325 4825
 	1    0    0    -1
 $EndComp
@@
 	9150 1025 9150 925
 $Comp
-L AA_vayuO2_symbols:PS2801-1 U8
-U 1 1 6165FCB0
+L AA_vayuO2_symbols:PS2801-4 U5
+U 4 1 6165FCB0
 P 7450 1425
-F 0 "U8" H 7475 1725 50  0000 C CNN
-F 1 "PS2801-1" H 7475 1625 40  0000 C CNN
-F 2 "AA_vayu:SO-4_5.3x2.7mm_P1.27mm" H 7450 1125 50  0001 C CIN
+F 0 "U5" H 7475 1725 50  0000 C CNN
+F 1 "PS2801-4" H 7475 1625 40  0000 C CNN
+F 2 "AA_vayu:SO-16_5.3x10.2mm_P1.27mm" H 7450 1125 50  0001 C CIN
 F 3 "" H 7425 1400 50  0001 L CNN
-	1    7450 1425
-	1    0    0    -1
-$EndComp
+	4    7450 1425
+	1    0    0    -1
+$EndComp
